File: AxoLights/axolights_leds.sch (KiCad schematic (older format))
At the start: 48 parts, among them Q1 BSS138, Q2 BSS138, Q3 BSS138, Q4 BSS138, Q5 BSS138, Q6 BSS138, Q7 BSS138, Q8 BSS138

Commit message: latest changes for production
Parts:
- removed D19, D20, D21: KA-3529ASELZ4S, myfootprint:LED-3528, symbol LED
- added D19, D20, D21: KA-3529ASELZ4S, symbol LED-RESCUE-axolights
- D1, D10, D11, D12, D13, D14, D15, D16, D17, D18, D2, D22, D23, D24, D3, D4, D5, D6, D7, D8, D9: symbol LED-RESCUE-axolights -> LED-RESCUE-axolights-RESCUE-axolights
Connections:
- net at D6.1 (A): now also D5.2 (K); no longer Q2.3 (D)
- net at D6.2 (K): now also Q2.3 (D); no longer D5.1 (K)
- net at R4.2: now also D4.1 (A); no longer D4.2 (A)
- net at D3.1 (A): now also D2.2 (K); no longer Q1.3 (D)
- net at D3.2 (K): now also Q1.3 (D); no longer D2.1 (K)
- net at R3.2: now also D1.1 (A); no longer D1.2 (A)
- net at D9.1 (A): now also D8.2 (K); no longer Q3.3 (D)
- net at D9.2 (K): now also Q3.3 (D); no longer D8.1 (K)
- net at R7.2: now also D7.1 (A); no longer D7.2 (A)
- net at D15.1 (A): now also D14.2 (K); no longer Q5.3 (D)
- net at D15.2 (K): now also Q5.3 (D); no longer D14.1 (K)
- net at R11.2: now also D13.1 (A); no longer D13.2 (A)
- net at D12.1 (A): now also D11.2 (K); no longer Q4.3 (D)
- net at D12.2 (K): now also Q4.3 (D); no longer D11.1 (K)
- net at R8.2: now also D10.1 (A); no longer D10.2 (A)
- net at D18.1 (A): now also D17.2 (K); no longer Q6.3 (D)
- net at D18.2 (K): now also Q6.3 (D); no longer D17.1 (K)
- net at R12.2: now also D16.1 (A); no longer D16.2 (A)
- net at R14.2: now also D19.2 (A)
- net at Q7.3 (D): now also D21.1 (K)
- net at D24.1 (A): now also D23.2 (K); no longer Q8.3 (D)
- net at D24.2 (K): now also Q8.3 (D); no longer D23.1 (K)
- net at R16.2: now also D22.1 (A); no longer D22.2 (A)
- new net: D4.2 (K), D5.1 (A)
- new net: D1.2 (K), D2.1 (A)
- new net: D7.2 (K), D8.1 (A)
- new net: D13.2 (K), D14.1 (A)
- new net: D10.2 (K), D11.1 (A)
- new net: D16.2 (K), D17.1 (A)
- new net: D22.2 (K), D23.1 (A)
- new net: D19.1 (K), D20.2 (A)
- new net: D20.1 (K), D21.2 (A)
Changed lines of the file:
@@
 $EndDescr
 $Comp
-L LED-RESCUE-axolights D6
+L LED-RESCUE-axolights-RESCUE-axolights D6
 U 1 1 58A971FA
 P 2000 6100
@@
 $EndComp
 $Comp
-L LED-RESCUE-axolights D5
+L LED-RESCUE-axolights-RESCUE-axolights D5
 U 1 1 58A971FF
 P 2000 5600
@@
 $EndComp
 $Comp
-L LED-RESCUE-axolights D4
+L LED-RESCUE-axolights-RESCUE-axolights D4
 U 1 1 58A97200
 P 2000 5100
@@
 $EndComp
 Wire Wire Line
-	10050 5700 10050 5300
+	10050 5300 10050 5700
 Wire Wire Line
-	10500 5700 10500 5300
+	10500 5300 10500 5700
 $Comp
 L BSS138 Q2
@@
 $EndComp
 Wire Wire Line
-	1700 6700 1250 6700
+	1250 6700 1700 6700
 Wire Wire Line
 	1500 6750 1500 6700
@@
 	2000 4400 2000 4500
 $Comp
-L LED-RESCUE-axolights D3
+L LED-RESCUE-axolights-RESCUE-axolights D3
 U 1 1 58A9720A
 P 1600 2700
@@
 	1600 3050 1600 2900
 $Comp
-L LED-RESCUE-axolights D2
+L LED-RESCUE-axolights-RESCUE-axolights D2
 U 1 1 58A9720F
 P 1600 2200
@@
 $EndComp
 $Comp
-L LED-RESCUE-axolights D1
+L LED-RESCUE-axolights-RESCUE-axolights D1
 U 1 1 58A97210
 P 1600 1700
@@
 $EndComp
 Wire Wire Line
-	1300 3300 850  3300
+	850  3300 1300 3300
 Wire Wire Line
 	1100 3350 1100 3300
@@
 	1600 1400 1600 1500
 $Comp
-L LED-RESCUE-axolights D9
+L LED-RESCUE-axolights-RESCUE-axolights D9
 U 1 1 58A97213
 P 3350 2700
@@
 	3350 3050 3350 2900
 $Comp
-L LED-RESCUE-axolights D8
+L LED-RESCUE-axolights-RESCUE-axolights D8
 U 1 1 58A97218
 P 3350 2200
@@
 $EndComp
 $Comp
-L LED-RESCUE-axolights D7
+L LED-RESCUE-axolights-RESCUE-axolights D7
 U 1 1 58A97219
 P 3350 1700
@@
 $EndComp
 Wire Wire Line
-	3050 3300 2600 3300
+	2600 3300 3050 3300
 Wire Wire Line
 	2850 3350 2850 3300
@@
 	3350 1400 3350 1500
 $Comp
-L LED-RESCUE-axolights D15
+L LED-RESCUE-axolights-RESCUE-axolights D15
 U 1 1 58A9721C
 P 5050 2700
@@
 $EndComp
 $Comp
-L LED-RESCUE-axolights D14
+L LED-RESCUE-axolights-RESCUE-axolights D14
 U 1 1 58A97221
 P 5050 2200
@@
 $EndComp
 $Comp
-L LED-RESCUE-axolights D13
+L LED-RESCUE-axolights-RESCUE-axolights D13
 U 1 1 58A97222
 P 5050 1700
@@
 $EndComp
 Wire Wire Line
-	4750 3300 4300 3300
+	4300 3300 4750 3300
 Wire Wire Line
 	4550 3350 4550 3300
@@
 	5050 1000 5050 1100
 $Comp
-L LED-RESCUE-axolights D12
+L LED-RESCUE-axolights-RESCUE-axolights D12
 U 1 1 58A97225
 P 3750 6050
@@
 $EndComp
 $Comp
-L LED-RESCUE-axolights D11
+L LED-RESCUE-axolights-RESCUE-axolights D11
 U 1 1 58A9722A
 P 3750 5550
@@
 $EndComp
 $Comp
-L LED-RESCUE-axolights D10
+L LED-RESCUE-axolights-RESCUE-axolights D10
 U 1 1 58A9722B
 P 3750 5050
@@
 $EndComp
 Wire Wire Line
-	3450 6650 3000 6650
+	3000 6650 3450 6650
 Wire Wire Line
 	3250 6700 3250 6650
@@
 	3750 4350 3750 4450
 $Comp
-L LED-RESCUE-axolights D18
+L LED-RESCUE-axolights-RESCUE-axolights D18
 U 1 1 58A9722E
 P 5450 6000
@@
 $EndComp
 $Comp
-L LED-RESCUE-axolights D17
+L LED-RESCUE-axolights-RESCUE-axolights D17
 U 1 1 58A97233
 P 5450 5500
@@
 $EndComp
 $Comp
-L LED-RESCUE-axolights D16
+L LED-RESCUE-axolights-RESCUE-axolights D16
 U 1 1 58A97234
 P 5450 5000
@@
 $EndComp
 Wire Wire Line
-	5150 6600 4700 6600
+	4700 6600 5150 6600
 Wire Wire Line
 	4950 6650 4950 6600
@@
 $EndComp
 Wire Wire Line
-	7400 3300 6950 3300
+	6950 3300 7400 3300
 Wire Wire Line
 	7200 3350 7200 3300
@@
 	7700 1000 7700 1100
 $Comp
-L LED-RESCUE-axolights D24
+L LED-RESCUE-axolights-RESCUE-axolights D24
 U 1 1 58A97240
 P 9950 2650
@@
 $EndComp
 $Comp
-L LED-RESCUE-axolights D23
+L LED-RESCUE-axolights-RESCUE-axolights D23
 U 1 1 58A97245
 P 9950 2150
@@
 $EndComp
 $Comp
-L LED-RESCUE-axolights D22
+L LED-RESCUE-axolights-RESCUE-axolights D22
 U 1 1 58A97246
 P 9950 1650
@@
 $EndComp
 Wire Wire Line
-	9650 3250 9200 3250
+	9200 3250 9650 3250
 Wire Wire Line
 	9450 3300 9450 3250
@@
 ED 65 30 18 8C 51 06 93 5E 06 83 C1 60 30 BE 50 58 9A 15 83 C1 60 30 18 5F 28 4C 7A 19 0C 06 83
 C1 F8 42 61 D2 CB 60 30 18 0C C6 17 0A 93 5E 06 83 C1 60 30 BE 50 FE 3F AB 46 48 5F BB 17 EF F9
-00 00 00 00 49 45 4E 44 AE 42 60 82 81
+00 00 00 00 49 45 4E 44 AE 42 60 82 82
 EndData
 $EndBitmap
@@
 69 67 67 F7 CC 50 03 18 63 06 96 A4 D9 86 4A A5 7A F0 E0 01 9F CF D7 79 BB 5A E8 A3 32 D3 F9 19
 D3 49 81 46 A3 D1 DE DE DE 26 14 8B 0F 33 1A 58 92 60 60 60 8C 08 78 33 02 06 06 C6 88 80 25 09
-06 06 C6 88 F8 FF 01 31 47 7E 68 65 D4 6D 96 00 00 00 00 49 45 4E 44 AE 42 60 82 90
+06 06 C6 88 F8 FF 01 31 47 7E 68 65 D4 6D 96 00 00 00 00 49 45 4E 44 AE 42 60 82 E4
 EndData
 $EndBitmap
@@
 60 34 32 A4 D1 50 28 14 72 B9 5C 83 77 9D B1 B1 31 85 42 D1 46 E5 51 84 19 01 91 24 04 04 04 1D
 02 71 95 44 40 40 D0 21 10 49 42 40 40 D0 21 10 49 42 40 40 D0 21 FE 3F F1 57 C2 52 63 5B 6A 1D
-00 00 00 00 49 45 4E 44 AE 42 60 82 61
+00 00 00 00 49 45 4E 44 AE 42 60 82 62
 EndData
 $EndBitmap
 $Comp
-L LED D19
-U 1 1 58AA4FCD
+L LED-RESCUE-axolights D19
+U 1 1 58C1E658
 P 7700 1700
 F 0 "D19" H 7700 1800 50  0000 C CNN
 F 1 "KA-3529ASELZ4S" V 7700 1250 50  0000 C CNN
-F 2 "myfootprint:LED-3528" H 7700 1700 50  0001 C CNN
+F 2 "" H 7700 1700 50  0000 C CNN
 F 3 "" H 7700 1700 50  0000 C CNN
 	1    7700 1700
@@
 $EndComp
 $Comp
-L LED D20
-U 1 1 58AA5288
+L LED-RESCUE-axolights D20
+U 1 1 58C1F0E7
 P 7700 2200
 F 0 "D20" H 7700 2300 50  0000 C CNN
 F 1 "KA-3529ASELZ4S" V 7700 1750 50  0000 C CNN
-F 2 "myfootprint:LED-3528" H 7700 2200 50  0001 C CNN
+F 2 "" H 7700 2200 50  0000 C CNN
 F 3 "" H 7700 2200 50  0000 C CNN
 	1    7700 2200
@@
 $EndComp
 $Comp
-L LED D21
-U 1 1 58AA5335
+L LED-RESCUE-axolights D21
+U 1 1 58C1F196
 P 7700 2700
 F 0 "D21" H 7700 2800 50  0000 C CNN
 F 1 "KA-3529ASELZ4S" V 7700 2250 50  0000 C CNN
-F 2 "myfootprint:LED-3528" H 7700 2700 50  0001 C CNN
+F 2 "" H 7700 2700 50  0000 C CNN
 F 3 "" H 7700 2700 50  0000 C CNN
 	1    7700 2700
